Commit message: Adding SLAM functionalities, MPC tests,...

File: ros_ws/src/my_robot_description/urdf/lidar.xacro (robot description, xacro)
@@ -1,14 +1,31 @@
 <?xml version="1.0"?>
 <robot xmlns:xacro="http://www.ros.org/wiki/xacro" >
-   <joint name="laser_joint" type="fixed">
-     <parent link="base_link"/>
-     <child link="laser_frame"/>
-     <origin xyz="0.1 0 ${base_height + 0.02}" rpy="0 0 0"/>
+   <link name="laser_frame"/>
+   <link name="mount_link">
+      <visual>
+         <geometry>
+               <box size="0.035 0.0646 0.039" />
+         </geometry>
+         <origin xyz="0 0 0" rpy="0 0 0" />
+         <material name="mycolor" />
+      </visual>
+      <collision>
+         <geometry>
+               <box size="0.035 0.0646 0.039" />
+         </geometry>
+         <origin xyz="0 0 0" rpy="0 0 0" />
+      </collision>
+      <xacro:box_inertia m="0.05" x="0.035" y="0.0646" z="0.039" o_xyz= "0 0 0.0195" o_rpy = "0 0 0"/>
+      </link>
+   <joint name="mount_joint" type="fixed">
+      <parent link="base_link"/>
+      <child link="mount_link"/>
+      <origin xyz="0.015 -0.0067 ${base_height+0.0195}" rpy= "0 0 0"/>
    </joint>
-   <link name="laser_frame">
+   <link name="laser_link">
       <visual>
          <origin xyz="0 0 0"/>
          <geometry>
-            <cylinder length="0.04" radius="0.05"/>
+            <cylinder length="0.034" radius="${0.035/2}"/>
          </geometry>
          <material name="laser_material">
@@ -19,32 +36,18 @@
          <origin xyz="0 0 0"/>
          <geometry>
-            <cylinder length="0.04" radius="0.05"/>
+            <cylinder length="0.034" radius="${0.035/2}"/>
          </geometry>
       </collision>
-      <xacro:cylinder_inertia m="0.1" r="0.05" l="0.04" o_xyz= "0 0 0" o_rpy= "0 0 0"/>
+      <xacro:cylinder_inertia m="0.15" r="${0.035/2}" l="0.034" o_xyz= "0 0 0" o_rpy= "0 0 0"/>
    </link>
-   <!-- 2D Lidar New Gazebo Sensor Plugin  -->
-   <gazebo reference="laser_frame">
-      <sensor name="laser" type="gpu_lidar">
-         <pose> 0 0 0 0 0 0 </pose>
-         <always_on>true</always_on>
-         <visualize>true</visualize>
-         <update_rate>10</update_rate>
-         <topic>scan</topic>
-         <gz_frame_id>laser_frame</gz_frame_id>
-         <lidar>
-            <scan>
-               <horizontal>
-               <samples>360</samples>
-               <min_angle>-3.14</min_angle>
-               <max_angle>3.14</max_angle>
-               </horizontal>
-            </scan>
-            <range>
-               <min>0.3</min>
-               <max>12</max>
-            </range>
-         </lidar>
-      </sensor>
-   </gazebo>
+    <joint name="laser_joint" type="fixed">
+     <parent link="mount_link"/>
+     <child link="laser_link"/>
+     <origin xyz="0 0 ${0.039/2 + 0.034/2}" rpy="0 0 0"/>
+   </joint>
+   <joint name="laser_frame_joint" type="fixed">
+      <parent link="laser_link"/>
+      <child link="laser_frame"/>
+      <origin xyz="0 0 ${0.026-0.034/2}" rpy="0 0 ${3.14159265/2}"/>
+   </joint>
 </robot>

File: ros_ws/src/my_robot_description/urdf/mobile_base.xacro (robot description, xacro)
@@ -13,5 +13,5 @@
             </geometry>
             <origin xyz="0 0 ${base_height / 2.0}" rpy="0 0 0" />
-            <material name="green" />
+            <material name="mycolor" />
         </visual>
         <collision>
@@ -21,5 +21,5 @@
             <origin xyz="0 0 ${base_height / 2.0}" rpy="0 0 0" />
         </collision>
-        <xacro:box_inertia m="5.0" x="${base_length}" y="${base_width}" z="${base_height}"
+        <xacro:box_inertia m="3.0" x="${base_length}" y="${base_width}" z="${base_height}"
                            o_xyz="0 0 ${base_height / 2.0}" o_rpy="0 0 0" />
     </link>
@@ -39,5 +39,5 @@
                 <origin xyz="0 0 0" rpy="0 0 0" />
             </collision>
-            <xacro:cylinder_inertia m="1.0" r="${wheel_radius}" l="${wheel_length}"
+            <xacro:cylinder_inertia m="0.2" r="${wheel_radius}" l="${wheel_length}"
                                     o_xyz="0 0 0" o_rpy="${pi / 2.0} 0 0" />
         </link>
@@ -59,5 +59,5 @@
             <origin xyz="0 0 0" rpy="0 0 0" />
         </collision>
-        <xacro:sphere_inertia m="0.5" r="${wheel_radius / 2.0}"
+        <xacro:sphere_inertia m="0.3" r="${wheel_radius / 2.0}"
                               o_xyz="0 0 0" o_rpy="0 0 0" />
     </link>
@@ -65,22 +65,22 @@
         <parent link="base_footprint" />
         <child link="base_link" />
-        <origin xyz="0 0 ${wheel_radius}" rpy="0 0 0" />
-    </joint>
-    <joint name="base_right_wheel_joint" type="continuous">
-        <parent link="base_link" />
-        <child link="right_wheel_link" />
-        <origin xyz="${-base_length / 4.0} ${-(base_width + wheel_length) / 2.0} 0" rpy="0 0 0" />
-        <axis xyz="0 1 0" />
-    </joint>
-    <joint name="base_left_wheel_joint" type="continuous">
-        <parent link="base_link" />
-        <child link="left_wheel_link" />
-        <origin xyz="${-base_length / 4.0} ${(base_width + wheel_length) / 2.0} 0" rpy="0 0 0" />
-        <axis xyz="0 1 0" />
+        <origin xyz="0 0 ${wheel_radius}" rpy="0 0 0"/>
     </joint>
     <joint name="base_caster_wheel_joint" type="fixed">
         <parent link="base_link" />
         <child link="caster_wheel_link" />
-        <origin xyz="${base_length / 3.0} 0 ${-wheel_radius / 2.0}" rpy="0 0 0" />
+        <origin xyz="${base_length / 3.0} 0 ${-wheel_radius / 2.0}" rpy="0 0 0"/>
+    </joint>
+    <joint name="base_right_wheel_joint" type="continuous">
+        <parent link="base_link"/>
+        <child link="right_wheel_link"/>
+        <origin xyz="${-base_length / 4.0} ${-(base_width + wheel_length) / 2.0} 0" rpy="0 0 0"/>
+        <axis xyz="0 1 0"/>
+    </joint>
+    <joint name="base_left_wheel_joint" type="continuous">
+        <parent link="base_link"/>
+        <child link="left_wheel_link"/>
+        <origin xyz="${-base_length / 4.0} ${(base_width + wheel_length) / 2.0} 0" rpy="0 0 0"/>
+        <axis xyz="0 1 0"/>
     </joint>
 </robot>

File: ros_ws/src/my_robot_description/urdf/my_robot.urdf.xacro (robot description, xacro)
@@ -3,6 +3,4 @@
 <xacro:include filename="$(find my_robot_description)/urdf/common_properties.xacro" />
 <xacro:include filename="$(find my_robot_description)/urdf/mobile_base.xacro" />
-<!--
 <xacro:include filename="$(find my_robot_description)/urdf/lidar.xacro" />
--->
 </robot>
